File: M7_sensor/M7_sensor.kicad_pcb (KiCad board)
At the start: 2 copper layers, 88.9 x 27.9 mm, 35 parts, among them J001 USB_OTG, J301 Battery_Cell, J401 CONN_01X16, J402 CONN_01X16, J403 CONN_01X16, J404 CONN_01X16, J405 CONN_01X06, J701 Micro_SD_Card_SPI, U201 MIC5319-3.3, U301 MCP73831, U401 TM4C1232, Y440 25MHz

Commit message: Adding Tomo
Parts:
- U401: value TM4C1232 -> ATSAMS70J
Connections:
- U401 pad 1: /1 -> Net-(U401-Pad1)
- U401 pad 10: /10 -> Net-(U401-Pad10)
- U401 pad 11: +3V3 -> Net-(U401-Pad11)
- U401 pad 12: GND -> Net-(U401-Pad12)
- U401 pad 13: /13 -> Net-(U401-Pad13)
- U401 pad 14: /14 -> Net-(U401-Pad14)
- U401 pad 15: /15 -> Net-(U401-Pad15)
- U401 pad 16: /16 -> Net-(U401-Pad16)
- U401 pad 17: /RX0 -> Net-(U401-Pad17)
- U401 pad 18: /TX0 -> Net-(U401-Pad18)
- U401 pad 19: /SCK0 -> Net-(U401-Pad19)
- U401 pad 2: +3V3 -> (no net)
- U401 pad 20: /CS_SD -> Net-(U401-Pad20)
- U401 pad 21: /MISO0 -> Net-(U401-Pad21)
- U401 pad 22: /MOSI0 -> Net-(U401-Pad22)
- U401 pad 23: /23 -> Net-(U401-Pad23)
- U401 pad 24: /24 -> Net-(U401-Pad24)
- U401 pad 25: /VDDC -> Net-(U401-Pad25)
- U401 pad 26: +3V3 -> Net-(U401-Pad26)
- U401 pad 27: GND -> Net-(U401-Pad27)
- U401 pad 28: /28 -> Net-(U401-Pad28)
- U401 pad 29: /29 -> Net-(U401-Pad29)
- U401 pad 3: GND -> Net-(U401-Pad3)
- U401 pad 30: /30 -> Net-(U401-Pad30)
- U401 pad 31: /31 -> Net-(U401-Pad31)
- U401 pad 32: /32 -> Net-(U401-Pad32)
- U401 pad 33: /33 -> Net-(U401-Pad33)
- U401 pad 34: /34 -> Net-(U401-Pad34)
- U401 pad 35: /35 -> Net-(U401-Pad35)
- U401 pad 36: /36 -> Net-(U401-Pad36)
- U401 pad 37: /37 -> Net-(U401-Pad37)
- U401 pad 38: /RESET -> Net-(U401-Pad38)
- U401 pad 39: GND -> Net-(U401-Pad39)
- U401 pad 4: /4 -> Net-(U401-Pad4)
- U401 pad 40: /OSC0 -> Net-(U401-Pad40)
- U401 pad 41: /OSC1 -> Net-(U401-Pad41)
- U401 pad 42: +3V3 -> Net-(U401-Pad42)
- U401 pad 43: /D- -> Net-(U401-Pad43)
- U401 pad 44: /D+ -> Net-(U401-Pad44)
- U401 pad 45: /45 -> Net-(U401-Pad45)
- U401 pad 46: /VBUS- -> Net-(U401-Pad46)
- U401 pad 47: /47 -> Net-(U401-Pad47)
- U401 pad 48: /48 -> Net-(U401-Pad48)
- U401 pad 49: /49 -> Net-(U401-Pad49)
- U401 pad 5: /5 -> Net-(U401-Pad5)
- U401 pad 50: /50 -> Net-(U401-Pad50)
- U401 pad 51: /51 -> Net-(U401-Pad51)
- U401 pad 52: /52 -> Net-(U401-Pad52)
- U401 pad 53: /53 -> Net-(U401-Pad53)
- U401 pad 54: +3V3 -> Net-(U401-Pad54)
- U401 pad 55: GND -> Net-(U401-Pad55)
- U401 pad 56: /VDDC -> Net-(U401-Pad56)
- U401 pad 57: /57 -> Net-(U401-Pad57)
- U401 pad 58: /58 -> Net-(U401-Pad58)
- U401 pad 59: /59 -> Net-(U401-Pad59)
- U401 pad 6: /6 -> Net-(U401-Pad6)
- U401 pad 60: /60 -> Net-(U401-Pad60)
- U401 pad 61: /61 -> Net-(U401-Pad61)
- U401 pad 62: /62 -> Net-(U401-Pad62)
- U401 pad 63: /63 -> Net-(U401-Pad63)
- U401 pad 64: /64 -> Net-(U401-Pad64)
- U401 pad 7: /7 -> Net-(U401-Pad7)
- U401 pad 8: /8 -> Net-(U401-Pad8)
- U401 pad 9: /9 -> Net-(U401-Pad9)
Routing:
- net +3V3: track 202.2 -> 0.00 mm, vias 10 -> 0
- net /D-: track 70.2 -> 0.00 mm, vias 2 -> 0
- net /D+: track 67.2 -> 0.00 mm, vias 4 -> 0
- net /VBUS+: track 66.4 -> 0.00 mm, vias 4 -> 0
- net /VDDC: track 58.8 -> 0.00 mm
- net /RX0: track 51.0 -> 0.00 mm
- net /TX0: track 48.1 -> 0.00 mm
- net /1: track 46.9 -> 0.00 mm, vias 1 -> 0
- net /63: track 45.0 -> 0.00 mm, vias 1 -> 0
- net /64: track 44.7 -> 0.00 mm, vias 1 -> 0
- net /33: track 43.8 -> 0.00 mm, vias 2 -> 0
- net /32: track 41.2 -> 0.00 mm
- net /35: track 39.8 -> 0.00 mm, vias 1 -> 0
- net /31: track 38.9 -> 0.00 mm
- net /34: track 38.9 -> 0.00 mm, vias 2 -> 0
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