File: Tomo/Tomo.kicad_pcb (KiCad board)
At the start: 2 copper layers, 35.6 x 55.9 mm, 62 parts, among them J001 USB_MICROB, J002 STANDOFF_GND, J101 Raspberry_Pi_1, J102 CONN_01X02, J301 CONN_02X03, J401 CONN_01X04, U001 FT232RL, U301 ADuM3221, U401 ATMEGA328P-AU, U501 MPU9250, U601 FGPMMOPA6H, U701 HMC5883L, U801 BMP180, U901 L3G4200D, X611 uFL, Y407 16MHz

Commit message: Rework to solve solder mask problem and use 1206 parts
Other:
- rule pad_to_mask_clearance: 0.2 -> 0
Changed lines of the file:
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@@
-(kicad_pcb (version 4) (host pcbnew 4.0.5+dfsg1-4)
+(kicad_pcb (version 20170123) (host pcbnew no-vcs-found-f042fcd~59~ubuntu17.04.1)
   (general
-    (links 188)
-    (no_connects 0)
-    (area 126.424999 98.544999 162.135001 154.575001)
     (thickness 1.6)
     (drawings 31)
@@
     (pad_size 5.4 5.4)
     (pad_drill 2.9)
-    (pad_to_mask_clearance 0.2)
+    (pad_to_mask_clearance 0)
     (aux_axis_origin 126.5 154.5)
     (visible_elements 7FFDFE7F)
@@
       (hpglpenspeed 20)
       (hpglpendiameter 15)
-      (hpglpenoverlay 2)
       (psnegative false)
       (psa4output false)
@@
   (module KwanSystems:FGPMMOPA6H (layer F.Cu)
     (at 135.81 116.154 270)
-    (fp_text reference U601 (at -8 -8.5 540) (layer F.SilkS) hide
+    (fp_text reference U601 (at -8 -8.5 180) (layer F.SilkS) hide
       (effects (font (size 0.9652 0.9652) (thickness 0.077216)) (justify left bottom))
     )
-    (fp_text value FGPMMOPA6H (at -8 9.5 540) (layer F.SilkS) hide
+    (fp_text value FGPMMOPA6H (at -8 9.5 180) (layer F.SilkS) hide
       (effects (font (size 0.77216 0.77216) (thickness 0.061772)) (justify left bottom))
     )
