File: Rocketometer055/Rocketometer055_pHAT.kicad_pcb (KiCad board)
At the start: 2 copper layers, 65 x 30 mm, 57 parts, among them J101 RPi_GPIO, J102 Micro_SD_Card_Det_Hirose_DM3AT, J601 USB_MICROB, J801 JST 2mm, Q650 PMOS, U101 LPC2148, U102 74CBTLV3257, U201 BME280, U301 BNO085, U401 ADXL375, U501 FGPMMOPA6H, U701 3.3V, U801 MCP73831, Y101 12MHz, Y301 32kiHz

Commit message: Started placing parts on Yukari6 hat
Parts:
- added C116: 100nF, KwanSystems:SMD_0402, F.Cu at (87.1, 18.0)
- J102: moved to B.Cu
- U102: footprint Housings_SOIC:SOIC-16_3.9x9.9mm_Pitch1.27mm -> Housings_SSOP:SSOP-16_3.9x4.9mm_Pitch0.635mm
- moved R804 276.9 mm to (10.9, -16.3)
- moved D801 276.5 mm to (10.9, -17.3)
- moved R801 275.2 mm to (13.0, -14.2), turned to 90 degrees
- moved U801 272.1 mm to (10.8, -14.2)
- moved D802 271.2 mm to (11.5, -10.4), turned to 270 degrees
- moved C803 271.2 mm to (11.4, -7.87)
- moved C802 270.8 mm to (14.0, -10.4), turned to 270 degrees
- moved C309 264.5 mm to (23.4, -3.81), turned to 90 degrees
- moved C303 263.1 mm to (25.7, -6.60)
- moved S701 261.8 mm to (10.9, -3.61), turned to 270 degrees
- moved C704 258.7 mm to (16.8, -5.84)
- moved C714 258.4 mm to (16.6, -1.27), turned to 180 degrees
- moved C326 258.0 mm to (31.0, -4.32)
- moved Y301 257.8 mm to (29.0, -4.32), turned to 270 degrees
- moved C715 257.4 mm to (19.1, -3.56), turned to 270 degrees
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- renumbered J801 to B801
Connections:
- B801 pad +: /Charger/VLIPO -> /VLIPO
- C803 pad 1: /Charger/VLIPO -> /VLIPO
- D802 pad 2: /Charger/VLIPO -> /VLIPO
- R101 pad 3: (no net) -> /SCL
- R101 pad 4: (no net) -> /SDA(BSL)
- R101 pad 5: (no net) -> VCC
- R101 pad 6: (no net) -> VCC
- R650 pad 1: /USB/USB_LIGHT+ -> /USB/CONN_D+
- R650 pad 2: /USB/USB_LIGHT+ -> /USB/USB_LIGHT-
- R650 pad 3: /USB/USB_LIGHT- -> /USB/USB_LIGHT+
- R650 pad 4: /USB/CONN_D+ -> /USB/USB_LIGHT+
- R651 pad 1: VCC -> /USB_ON
- R651 pad 2: /USB_ON -> VCC
- R651 pad 3: /VBUS -> /USB_SOFTCONNECT
- R651 pad 4: /USB_SOFTCONNECT -> /VBUS
- U102 pad 15: VCC -> GND
- U501 pad 4: /GPS/VBACKUP -> /VLIPO
- U801 pad 3: /Charger/VLIPO -> /VLIPO
Routing:
- net /VBUS: track 0.00 -> 43.1 mm, vias 0 -> 1
- net /PI_TX: track 0.00 -> 31.4 mm, vias 0 -> 1
- net /S: track 0.00 -> 14.4 mm
- net VCC: track 0.00 -> 13.3 mm
- net /VRAW: track 0.00 -> 8.88 mm
- net /LPC_TX0(PWMR): track 0.00 -> 8.37 mm
- net /VLIPO: track 0.00 -> 8.32 mm
- net /LPC_RX0: track 0.00 -> 6.69 mm
- net /USBD+: track 0.00 -> 6.19 mm
- net /XTAL2: track 0.00 -> 5.40 mm
- net /USBD-: track 0.00 -> 5.13 mm
- net /USB_SOFTCONNECT: track 0.00 -> 5.00 mm
- net /XTAL1: track 0.00 -> 3.50 mm
- net /USB/CONN_D+: track 0.00 -> 2.60 mm
- net /Charger/STAT-: track 0.00 -> 2.26 mm
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Other:
- net class VBUS added: clearance 0.1524, trace_width 0.508, via_dia 0.508, via_drill 0.254
