File: YukariWheel/YukariWheel.kicad_pcb (KiCad board)
At the start: 2 copper layers, 55.9 x 22.9 mm, 23 parts, among them J001 USB_MICROB, J301 JST 2mm, J401 M07, J701 Micro_SD_Card_Det_Hirose_DM3AT, U401 LPC2148

Commit message: Started layout on YukariWheel
Parts:
- removed C443: 100nF, KwanSystems:SMD_0402
- removed D050: BLUE, LED-0603
- removed D301: YELLOW, LED-0603
- removed D401: HSMF-C118, HSMF-C118
- removed J001: USB_MICROB, UB-MC5BR3-SD204-4S
- removed J401: M07, 1X08
- removed J701: Micro_SD_Card_Det_Hirose_DM3AT, MICROSD-SOCKET-PP
- removed JP1, JP2, JP3, JP4, JP5: STAND-OFFTIGHT, STAND-OFF-TIGHT
- removed S201: SPDT, AYZ0202
- removed S456: SOLDERJUMPERNO, SJ_2S-NO
- removed S457: SPST, B3U-1000P
- removed S458: B3U-1000P, B3U-1000P
- removed U$1, U$5: , KWAN_ACC
- removed U$4: , AXES
- removed U$6: , OSHW_ACC
- added C105: 100nF, KwanSystems:SMD_0402, F.Cu at (163.2, 111.4)
- added C111: 33pF, KwanSystems:SMD_0402, F.Cu at (161.5, 117.8)
- added C112: 33pF, KwanSystems:SMD_0402, F.Cu at (166.3, 119.1)
- added C117: 100nF, KwanSystems:SMD_0402, F.Cu at (169.1, 118.5)
- added C140: 1uF, KwanSystems:SMD_0402, F.Cu at (170.1, 107.1)
- added C201: 1uF, KwanSystems:SMD_0402, F.Cu at (109.4, 47.7)
- added C204: 100nF, KwanSystems:SMD_0402, F.Cu at (104.1, 47.7)
- added C205: 4.7nF, KwanSystems:SMD_0402, F.Cu at (104.8, 47.7)
- added C301: 100nF, KwanSystems:SMD_0402, F.Cu at (135.3, 143.7)
- added C305: 100nF, KwanSystems:SMD_0402, F.Cu at (135.3, 134.0)
- added C308: 10uF, KwanSystems:SMD_0402, F.Cu at (135.3, 133.3)
- added C401: 1uF, KwanSystems:SMD_0402, F.Cu at (109.4, 44.1)
- added C404: 100nF, KwanSystems:SMD_0402, F.Cu at (104.1, 44.1)
- added C803: 100nF, KwanSystems:SMD_0402, F.Cu at (150.5, 139.1)
- added C809: 100nF, KwanSystems:SMD_0402, F.Cu at (148.5, 140.6)
- added C825: 120nF, KwanSystems:SMD_0402, F.Cu at (154.1, 139.1)
- added C826: 22pF, KwanSystems:R_Array_Convex_2x0402, F.Cu at (155.9, 141.6)
- added C828: 6.8nF, KwanSystems:SMD_0402, F.Cu at (154.1, 139.9)
- added J101: Conn_01x08, Pin_Headers:Pin_Header_Straight_1x08_Pitch2.54mm, F.Cu at (135.2, 109.1)
- added J102: CONN_01X02, Socket_Strips:Socket_Strip_Straight_1x02_Pitch2.54mm, F.Cu at (163.9, 123.2)
- added L201: Ferrite_Bead_Small, KwanSystems:SMD_0603, F.Cu at (110.7, 47.7)
- added L401: Ferrite_Bead_Small, KwanSystems:SMD_0603, F.Cu at (110.7, 44.1)
- added R001: 196, KwanSystems:SMD_1206, F.Cu at (111.8, 98.9)
- added R003: 10k, KwanSystems:SMD_1206, F.Cu at (111.8, 101.0)
- added R101: 196, KwanSystems:SMD_1206, F.Cu at (98.7, 88.1)
- added R102: 10k, KwanSystems:R_Array_Convex_4x0402, F.Cu at (167.6, 105.8)
- added R103: 10k, KwanSystems:SMD_1206, F.Cu at (101.0, 88.1)
- added R117: 10k, KwanSystems:SMD_0402, F.Cu at (164.0, 121.3)
- added S157: SPST, KwanSystems:SW_SPST_B3U-1000P, F.Cu at (162.2, 114.2)
- added S401: SPDT, KwanSystems:SWITCH_DPDT_AZY0202, F.Cu at (107.1, 39.0)
- added U000: EE-SY199, KwanSystems:EE-SY199, B.Cu at (111.8, 100.0)
- added U001: Designed_With_Kicad, Symbols:Symbol_KiCAD-Logo_CopperAndSilkScreenTop, B.Cu at (101.0, 43.6)
- added U002: KwanSystems, KwanSystems:KWAN_CIRCLE_soldermask, F.Cu at (98.7, 39.8)
- added U100: EE-SY199, KwanSystems:EE-SY199, B.Cu at (100.0, 88.2)
- added U101: LPC2103, Housings_QFP:LQFP-48_7x7mm_Pitch0.5mm, F.Cu at (169.4, 112.8)
- added U201: 1.8V, TO_SOT_Packages_SMD:SOT-23-5, F.Cu at (107.0, 47.7)
- added U301: ADuM3221, SMD_Packages:SOIC-8-N, F.Cu at (135.3, 138.9)
- added U801: BNO055, KwanSystems:BNO055, F.Cu at (150.9, 142.2)
- added Y101: 12MHz, Crystals:Crystal_SMD_Abracon_ABM8G-4pin_3.2x2.5mm, F.Cu at (163.9, 117.9)
- added Y801: 32kiHz, Crystals:Crystal_SMD_2012-2pin_2.0x1.2mm, F.Cu at (154.1, 141.7)
- C405: value 18pF -> 4.7nF
- J301: value JST 2mm -> CONN_02X03; footprint JST-2-SMD -> Pin_Headers:Pin_Header_Straight_2x03_Pitch2.54mm
- U401: value LPC2148 -> 3.3V; footprint Housings_QFP:LQFP-64_10x10mm_Pitch0.5mm -> TO_SOT_Packages_SMD:SOT-23-5
- moved J301 84.8 mm to (113.5, 37.0), turned to 0 degrees
- moved C405 78.4 mm to (104.8, 44.1), turned to 90 degrees
- moved U401 70.9 mm to (107.0, 44.1)
Connections:
- C405 pad 1: GND -> /3V3+
- C405 pad 2: /RTXC2 -> GND
- J301 pad 1: GND -> /STEER_HI
- J301 pad 2: /VLIPO -> /THROTTLE_HI
- U401 pad 1: Net-(U401-Pad1) -> /VBAT-
- U401 pad 2: Net-(U401-Pad2) -> GND
- U401 pad 3: /RTXC1 -> /Regulator3V3/PWR_EN
- U401 pad 4: Net-(U401-Pad4) -> /Regulator3V3/BYP
- U401 pad 5: /RTXC2 -> /3V3+
Routing:
- net +3V3: track 0.00 -> 62.8 mm
- net /ENC0: track 0.00 -> 14.9 mm, vias 0 -> 1
- net /ENC1: track 0.00 -> 11.3 mm, vias 0 -> 1
- net /RST: track 0.00 -> 10.3 mm
- net +BATT: track 0.00 -> 10.1 mm
- net /3V3+: track 0.00 -> 9.65 mm
- net /CS0: track 6.94 -> 0.00 mm, vias 1 -> 0
- net /XTAL1: track 0.00 -> 6.63 mm
- net /VBAT-: track 0.00 -> 5.94 mm
- net /SDA: track 0.00 -> 4.87 mm
- net /SCL: track 0.00 -> 4.11 mm
- net /BNO055/XOUT32: track 0.00 -> 3.83 mm
- net /D0: track 0.00 -> 3.76 mm, vias 0 -> 1
- net /D1: track 0.00 -> 3.65 mm, vias 0 -> 1
- net /XTAL2: track 0.00 -> 3.64 mm
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Other:
- board size 55.9 x 22.9 mm -> 24 x 71 mm
- board text added: "0"
- board text added: "1"
- board text added: "24 Jul 2017"
- board text added: "Tomo Encoder 1.1"
- board text added: "github.com/kwan3217"
- board text removed: "3V3"
- board text removed: "Acc/Gyro"
- board text removed: "BSL"
- board text removed: "Baro"
- board text removed: "Boot"
- board text removed: "Compass"
- board text removed: "D"
- board text removed: "GND"
- board text removed: "HighAcc"
- board text removed: "Kwan Systems"
- board text removed: "On"
- board text removed: "RX0"
- board text removed: "Reset"
- board text removed: "RocketometerMPU6050"
- board text removed: "SCL"
- board text removed: "SDA"
- board text removed: "St Kwan's Home for"
- board text removed: "TX0"
- board text removed: "VBUS"
- board text removed: "a division of"
- board text removed: "stkwans.blogspot.com"
- board text removed: "the Terminally ADD"
- board text removed: "v1.0 19 Nov 2012"

Commit message: More layout of YukariWheel
Parts:
- moved C117 98.4 mm to (103.6, 45.1), turned to 180 degrees
- moved C112 95.6 mm to (106.3, 44.6), turned to 270 degrees
- moved J102 94.0 mm to (96.2, 58.1)
- moved C825 92.0 mm to (115.0, 55.8)
- moved C826 92.0 mm to (116.8, 58.2)
- moved Y801 92.0 mm to (115.0, 58.3)
- moved C803 92.0 mm to (111.4, 55.8)
- moved U801 92.0 mm to (111.8, 58.9)
- moved C809 92.0 mm to (109.4, 57.3)
- moved C828 92.0 mm to (115.0, 56.6)
- moved C305 91.2 mm to (115.0, 45.1)
- moved C308 91.2 mm to (115.0, 44.4)
- moved C301 91.2 mm to (115.0, 54.8)
- moved U301 91.2 mm to (115.0, 50.0)
- moved Y101 90.8 mm to (108.7, 45.8), turned to 180 degrees
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Routing:
- net +BATT: track 10.1 -> 20.7 mm, vias 0 -> 1
- net +3V3: track 62.8 -> 68.4 mm
- net /THROTTLE_HI: track 0.00 -> 5.61 mm
- net /STEER_HI: track 0.00 -> 4.91 mm
- net /3V3+: track 9.65 -> 6.79 mm

Commit message: Continuing layout of YukariWheel
Routing:
- net +1V8: track 3.05 -> 32.7 mm, vias 0 -> 2
- net /SDA: track 4.87 -> 27.9 mm, vias 0 -> 1
- net /SCL: track 4.11 -> 27.2 mm, vias 0 -> 3
- net /STEERING: track 0.00 -> 18.7 mm, vias 0 -> 2
- net /ACCINT: track 0.00 -> 14.6 mm, vias 0 -> 2
- net /TX0: track 0.00 -> 12.9 mm
- net /ENC0: track 14.9 -> 3.41 mm
- net /RX0: track 0.00 -> 11.4 mm
- net /BSL: track 2.26 -> 11.7 mm, vias 0 -> 1
- net +3V3: track 68.4 -> 59.8 mm, vias 0 -> 2
- net /ENC1: track 11.3 -> 3.65 mm
- net /THROTTLE: track 0.00 -> 7.51 mm
- net /GO_BTN: track 0.00 -> 2.08 mm
Other:
- board text removed: "+"
- board text removed: "-"
