File: M7_055/M7_055.kicad_pcb (KiCad board)
At the start: 2 copper layers, 48 parts, among them J101 USB_MICROB, J801 Micro_SD_Card_Det_Hirose_DM3AT, U101 STM32F722, U201 BNO055, U301 FGPMMOPA6H, U401 BME280, U501 ADXL375, U601 MCP73831, U701 3.3V, X311 uFL, Y201 32kiHz

Commit message: More work on M7_055
Parts:
- added C105: 22pF, KwanSystems:R_Array_Convex_2x0402, F.Cu at (185.7, 109.0)
- added J102: Conn_01x08, Pin_Headers:Pin_Header_Straight_1x08_Pitch2.54mm, F.Cu at (171.7, 67.1)
- added R107: 10k, KwanSystems:R_Array_Convex_4x0402, F.Cu at (195.3, 101.8)
- added S107: SW_SPST, KwanSystems:SW_SPST_B3U-1000P, F.Cu at (173.2, 107.7)
- added S160: SW_SPST, KwanSystems:SW_SPST_B3U-1000P, F.Cu at (180.6, 126.5)
- added Y101: Crystal_GND24, Crystals:Crystal_SMD_3225-4pin_3.2x2.5mm, F.Cu at (188.5, 108.7)
- moved C119 28.7 mm to (194.1, 118.1), turned to 180 degrees
- moved C113 27.5 mm to (189.7, 112.8), turned to 90 degrees
- moved C164 22.3 mm to (193.5, 103.6)
- moved C130 21.0 mm to (198.9, 118.1)
- moved C112 17.4 mm to (188.5, 112.8), turned to 90 degrees
- moved C148 14.7 mm to (204.2, 106.9), turned to 270 degrees
- moved C118 11.2 mm to (194.1, 119.4), turned to 180 degrees
- moved C132 6.83 mm to (201.7, 118.1), turned to 180 degrees
Connections:
- net Net-(C130-Pad1) renamed /VCAP
- U101 pad 14: (no net) -> /BNO_INT
- U101 pad 15: (no net) -> /ADXL_INT
- U101 pad 16: (no net) -> /GPS_PPS
- U101 pad 17: (no net) -> /GPS_FIX
- U101 pad 28: (no net) -> /M7_TX
- U101 pad 29: (no net) -> /M7_RX
- U101 pad 5: (no net) -> /XIN
- U101 pad 6: (no net) -> /XOUT
- U101 pad 60: (no net) -> /BOOT
- U101 pad 7: (no net) -> /RESET
- U201 pad 14: (no net) -> /BNO_INT
- U301 pad 13: (no net) -> /GPS_PPS
- U301 pad 5: (no net) -> /GPS_FIX
- U501 pad 8: (no net) -> /ADXL_INT
Routing:
- net +3V3: track 40.3 -> 67.1 mm
- net /RESET: track 0.00 -> 10.9 mm
- net /XIN: track 0.00 -> 6.75 mm
- net /XOUT: track 0.00 -> 6.17 mm
- net /SCL: track 0.00 -> 2.92 mm
- net /SDA: track 0.00 -> 2.87 mm
- net /BOOT: track 0.00 -> 2.87 mm
- net /VCAP: track 0.00 -> 2.57 mm

Commit message: Pushing
Parts:
- removed S701: SPDT, KwanSystems:SWITCH_DPDT_AZY0202
- added D137: HSMF-C118, KwanSystems:HSMF-C118, F.Cu at (164.8, 78.2)
- C801, J801, U301: moved to B.Cu
- J102: value Conn_01x08 -> Conn_01x12; footprint Pin_Headers:Pin_Header_Straight_1x08_Pitch2.54mm -> Pin_Headers:Pin_Header_Straight_1x12_Pitch2.54mm
- moved J801 269.0 mm to (30.4, -20.5)
- moved C226 261.6 mm to (12.4, -7.62)
- moved C228 261.6 mm to (12.4, -11.2)
- moved C506 261.6 mm to (7.87, -18.5)
- moved R506 261.6 mm to (5.59, -15.7)
- moved U201 261.6 mm to (9.14, -9.14)
- moved U501 261.6 mm to (9.14, -15.0)
- moved C203 261.6 mm to (9.14, -12.4)
- moved C209 261.6 mm to (6.35, -10.5)
- moved C225 261.6 mm to (12.4, -12.4)
- moved C406 261.6 mm to (6.60, -5.08)
- moved C501 261.6 mm to (10.4, -17.3)
- moved C505 261.6 mm to (7.87, -17.3)
- moved U401 261.6 mm to (9.18, -4.80)
- moved Y201 261.6 mm to (12.4, -9.40)
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Connections:
- B304 pad +: /GPS/VBACKUP -> /VBAT
- C112 pad 1: +3V3 -> GND
- C112 pad 2: GND -> +3V3
- C113 pad 1: +3V3 -> GND
- C113 pad 2: GND -> +3V3
- C118 pad 1: +3V3 -> GND
- C118 pad 2: GND -> +3V3
- C119 pad 1: +3V3 -> GND
- C119 pad 2: GND -> +3V3
- C130 pad 1: /VCAP -> GND
- C130 pad 2: GND -> /VCAP
- C132 pad 1: +3V3 -> GND
- C132 pad 2: GND -> +3V3
- C148 pad 1: +3V3 -> GND
- C148 pad 2: GND -> +3V3
- C164 pad 1: +3V3 -> GND
- C164 pad 2: GND -> +3V3
- C304 pad 1: /GPS/VBACKUP -> /VBAT
- J101 pad 2: (no net) -> /D-
- J101 pad 3: (no net) -> /D+
- J801 pad 2: (no net) -> /CS_uSD
- J801 pad 3: (no net) -> /MOSI
- J801 pad 5: +3V3 -> /SCK
- J801 pad 7: +3V3 -> /MISO
- R107 pad 1: +3V3 -> /RESET
- R107 pad 8: /RESET -> +3V3
- R304 pad 1: /GPS/VBACKUP -> /VBAT
- S107 pad 1: GND -> /RESET
- S107 pad 2: /RESET -> GND
- S160 pad 1: /BOOT -> +3V3
- S160 pad 2: +3V3 -> /BOOT
- U101 pad 1: +3V3 -> /VBAT
- U101 pad 14: /BNO_INT -> (no net)
- U101 pad 28: /M7_TX -> /GPS_RX
- U101 pad 29: /M7_RX -> /GPS_TX
- U101 pad 37: (no net) -> /PWMR
- U101 pad 38: (no net) -> /PWMG
- U101 pad 39: (no net) -> /PWMB
- U101 pad 40: (no net) -> /PWM4
- U101 pad 42: /GPS_RX -> /M7_TX
- U101 pad 43: /GPS_TX -> /M7_RX
- U101 pad 44: (no net) -> /D-
- U101 pad 45: (no net) -> /D+
- U101 pad 50: (no net) -> /BNO_INT
- U101 pad 54: (no net) -> /CS_uSD
- U101 pad 55: (no net) -> /SCK
- U101 pad 56: (no net) -> /MISO
- U101 pad 57: (no net) -> /MOSI
- U301 pad 4: /GPS/VBACKUP -> /VBAT
- Y101 pad 1: GND -> /XOUT
- Y101 pad 2: /XIN -> GND
- Y101 pad 3: GND -> /XIN
- Y101 pad 4: /XOUT -> GND
Routing:
- net /SCL: track 2.92 -> 27.3 mm, vias 0 -> 3
- net /BNO_INT: track 0.00 -> 24.2 mm, vias 0 -> 2
- net /SDA: track 2.87 -> 22.4 mm, vias 0 -> 2
- net /RESET: track 10.9 -> 0.00 mm
- net /MISO: track 0.00 -> 9.80 mm, vias 0 -> 1
- net /Regulator/VIN: track 13.9 -> 23.8 mm
- net /SCK: track 0.00 -> 8.64 mm, vias 0 -> 1
- net /CS_uSD: track 0.00 -> 5.73 mm, vias 0 -> 1
- net /Regulator/PWR_EN: track 2.18 -> 7.80 mm
- net /MOSI: track 0.00 -> 5.39 mm, vias 0 -> 1
- net +3V3: track 67.1 -> 61.8 mm, vias 0 -> 1
- net GND: track 1.95 -> 3.19 mm
Other:
- board outline added: 55.9 x 22.9 mm

Commit message: Baseline routing completed
Parts:
- removed B304: Coin_Cell, KwanSystems:CR1220-2
- removed C304: 220mF, KwanSystems:Supercap
- removed D304: D_Schottky, KwanSystems:D_0603
- removed R304: 10k, KwanSystems:SMD_0603
- added J103: STANDOFF_GND, KwanSystems:MountingHole_2.9mm_M2.5_Pad, F.Cu at (2.54, -2.54)
- added J104: STANDOFF_GND, KwanSystems:MountingHole_2.9mm_M2.5_Pad, F.Cu at (2.54, -20.3)
- added J105: STANDOFF_GND, KwanSystems:MountingHole_2.9mm_M2.5_Pad, F.Cu at (53.3, -20.3)
- added J106: STANDOFF_GND, KwanSystems:MountingHole_2.9mm_M2.5_Pad, F.Cu at (53.3, -2.54)
- added R137: 68, KwanSystems:R_Array_Convex_4x0402, F.Cu at (16.8, -9.14)
- added REF**: StKwans, KwanSystems:StKwans, F.Cu at (26.9, -17.8)
- added S701: SPDT, KwanSystems:SW_SPST_CJS120xA, F.Cu at (46.9, -2.54)
- C105, C112, C113, C118, C119, C130, C132, C148, C164, C225, C506, R107, R506, U101: moved to B.Cu
- C303: footprint KwanSystems:SMD_1206 -> KwanSystems:SMD_0603_pol
- J102: value Conn_01x12 -> Conn_01x16; footprint Pin_Headers:Pin_Header_Straight_1x12_Pitch2.54mm -> Pin_Headers:Pin_Header_Straight_1x16_Pitch2.54mm; moved to B.Cu
- U301: moved to F.Cu
- Y101: value Crystal_GND24 -> 12MHz; moved to B.Cu
- moved X311 197.0 mm to (20.1, -2.29)
- moved C301 191.5 mm to (38.9, -16.8), turned to 90 degrees
- moved C303 190.3 mm to (40.1, -16.8), turned to 270 degrees
- moved J102 188.6 mm to (8.89, -21.6), turned to 270 degrees
- moved L301 186.3 mm to (42.4, -17.5), turned to 180 degrees
- moved D137 173.2 mm to (16.8, -11.7)
- moved U301 39.1 mm to (29.6, -9.52), turned to 270 degrees
- moved C148 18.7 mm to (25.9, -1.26), turned to 0 degrees
- moved C801 17.8 mm to (9.65, -1.52)
- moved C105 17.6 mm to (28.8, -17.8), turned to 90 degrees
- moved C132 14.3 mm to (38.4, -3.79), turned to 270 degrees
- moved Y101 12.8 mm to (28.9, -15.4)
- moved C112 12.8 mm to (32.5, -15.5)
- moved C113 10.5 mm to (32.5, -14.2)
- moved C130 9.40 mm to (38.4, -6.58)
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Connections:
- net /Sheet5A4D5668/VBUS renamed /VBUS
- C303 pad 1: GND -> /GPS/VGPS
- C303 pad 2: /GPS/VGPS -> GND
- C701 pad 1: /Regulator/VIN -> /VRAW
- D137 pad 2: /PWMR -> /PWMR-
- D137 pad 3: /PWMG -> /PWMG-
- D137 pad 4: /PWMB -> /PWMB-
- D602 pad 3: /Regulator/VIN -> /VRAW
- J102 pad 10: /PWMB -> /GPS_RX
- J102 pad 11: /PWMG -> /GPS_TX
- J102 pad 12: /PWMR -> /M7_RX
- J102 pad 2: /BOOT -> /PWMB
- J102 pad 3: /RESET -> /PWMG
- J102 pad 4: /M7_TX -> /PWMR
- J102 pad 5: /M7_RX -> GND
- J102 pad 8: +3V3 -> /BOOT
- J102 pad 9: /PWM4 -> /RESET
- R107 pad 1: /RESET -> (no net)
- R107 pad 3: /SDA -> /SCL
- R107 pad 4: /SCL -> /SDA
- R107 pad 8: +3V3 -> (no net)
- U101 pad 1: /VBAT -> +3V3
- U101 pad 40: /PWM4 -> (no net)
- U301 pad 4: /VBAT -> /VRAW
- U701 pad 1: /Regulator/VIN -> /VRAW
- Y101 pad 2: GND -> (no net)
Routing:
- net +3V3: track 61.8 -> 163.8 mm, vias 1 -> 10
- net GND: track 3.19 -> 51.2 mm, vias 2 -> 9
- net /PWMR: track 0.00 -> 43.4 mm, vias 0 -> 2
- net /PWMG: track 0.00 -> 36.5 mm, vias 0 -> 2
- net /PWMB: track 0.00 -> 35.4 mm, vias 0 -> 2
- net /ADXL_INT: track 0.00 -> 35.0 mm, vias 0 -> 1
- net /RESET: track 0.00 -> 34.4 mm, vias 0 -> 3
- net /D+: track 0.00 -> 32.9 mm, vias 0 -> 1
- net /D-: track 0.00 -> 32.3 mm, vias 0 -> 1
- net /GPS_TX: track 0.00 -> 32.2 mm, vias 0 -> 1
- net /GPS_RX: track 0.00 -> 31.9 mm, vias 0 -> 1
- net /VRAW: track 0.00 -> 30.1 mm
- net /M7_RX: track 0.00 -> 27.8 mm, vias 0 -> 5
- net /M7_TX: track 0.00 -> 27.2 mm, vias 0 -> 5
- net /SDA: track 22.4 -> 48.1 mm, vias 2 -> 4
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- added copper zone on B.Cu, net GND
- added copper zone on F.Cu, net GND

Commit message: Starting IOIO_Sensinator
Parts:
- removed X311: uFL, KwanSystems:U.FL
- added R174: 5.1k, KwanSystems:R_Array_Convex_2x0402, F.Cu at (47.0, -8.22)
- C603, D602, R601, R604, U601: moved to B.Cu
- J101: value USB_MICROB -> USB_C2; footprint KwanSystems:USB_Micro-B_Molex_47346-0001 -> KwanSystems:MolexUSBTypeC2
- moved C602 11.2 mm to (43.2, -2.55)
- moved C705 8.22 mm to (44.5, -7.60)
- moved R601 5.80 mm to (44.5, -8.89), turned to 180 degrees
- moved R604 3.31 mm to (44.5, -15.2)
- moved C701 3.06 mm to (44.5, -14.0), turned to 180 degrees
- moved C704 3.06 mm to (44.5, -8.89), turned to 0 degrees
- moved U701 3.05 mm to (44.5, -11.4), turned to 270 degrees
- moved D602 2.97 mm to (44.5, -6.60), turned to 90 degrees
- moved D601 2.81 mm to (44.5, -15.2)
- moved U601 2.79 mm to (44.5, -11.4), turned to 270 degrees
- moved C603 2.54 mm to (44.5, -14.0), turned to 180 degrees
- moved L301 0.92 mm to (41.9, -16.8), turned to 90 degrees
- turned J101 to 90 degrees
Connections:
- J101 pad 4: (no net) -> /CC2
Routing:
- net +3V3: track 163.8 -> 193.9 mm
- net /VBUS: track 13.1 -> 37.2 mm, vias 0 -> 2
- net /CC2: track 0.00 -> 14.6 mm
- net /VRAW: track 30.1 -> 42.7 mm, vias 0 -> 1
- net /D+: track 32.9 -> 41.8 mm, vias 1 -> 2
- net /Sheet5A4D5668/VLIPO: track 10.4 -> 16.4 mm, vias 1 -> 0
- net /CC1: track 0.00 -> 5.74 mm, vias 0 -> 2
- net GND: track 51.2 -> 46.1 mm, vias 9 -> 8
- net /D-: track 32.3 -> 36.2 mm
- net /Sheet5A4D5668/STAT-: track 3.69 -> 0.00 mm
- net /Regulator/PWR_EN: track 10.3 -> 11.8 mm
- net /GPS/ANT: track 1.34 -> 0.38 mm
- net /Sheet5A4D5668/STAT+: track 1.54 -> 1.44 mm, vias 0 -> 1
Other:
- board text added: "3V3"
- board text added: "BT"
- board text added: "GND"
- board text added: "GRX"
- board text added: "GTX"
- board text added: "PWB"
- board text added: "PWG"
- board text added: "PWR"
- board text added: "RST"
- board text added: "RX"
- board text added: "SCL"
- board text added: "SDA"
- board text added: "TX"
