File: ioio_sensinator/ioio_sensinator.kicad_pcb (KiCad board)
At the start: 2 copper layers, 37 parts, among them U201 MPU9250, U301 FGPMMOPA6H, U401 ADXL375, U501 BNO055, U601 BME280, X311 uFL, Y501 32kiHz

Commit message: More wiring of ioio_sensinator
Parts:
- added REF**: STANDOFF_NONPLATED, KwanSystems:STANDOFF_NONPLATED, F.Cu at (2.54, -2.54)
- added REF**: STANDOFF_NONPLATED, KwanSystems:STANDOFF_NONPLATED, F.Cu at (2.54, -27.9)
- added REF**: STANDOFF_NONPLATED, KwanSystems:STANDOFF_NONPLATED, F.Cu at (66.0, -27.9)
- added REF**: STANDOFF_NONPLATED, KwanSystems:STANDOFF_NONPLATED, F.Cu at (66.0, -2.54)
- moved U201 192.0 mm to (17.2, -8.14)
- moved X311 190.1 mm to (34.3, -5.08), turned to 90 degrees
- moved U301 181.6 mm to (41.0, -18.9), turned to 270 degrees
- moved C304 180.0 mm to (61.0, -17.8)
- moved B304 179.9 mm to (61.0, -17.8), turned to 180 degrees
- moved C303 176.7 mm to (51.6, -26.4), turned to 180 degrees
- moved L301 171.7 mm to (51.3, -22.6), turned to 180 degrees
- moved D304 167.8 mm to (55.6, -24.4), turned to 180 degrees
- moved C301 167.2 mm to (51.6, -24.4), turned to 180 degrees
- moved R304 165.0 mm to (55.6, -22.9)
- moved U501 161.9 mm to (25.4, -22.9)
- moved C503 158.0 mm to (25.4, -26.2)
- moved C406 157.0 mm to (11.7, -17.8), turned to 270 degrees
- moved C509 156.7 mm to (22.6, -24.4), turned to 90 degrees
- moved C526 155.2 mm to (31.0, -22.6)
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Connections:
- JP20 pad 1: (no net) -> Net-(JP20-Pad1)
- JP20 pad 10: (no net) -> /GPS_RX
- JP20 pad 11: (no net) -> Net-(JP20-Pad11)
- JP20 pad 12: (no net) -> Net-(JP20-Pad12)
- JP20 pad 13: (no net) -> Net-(JP20-Pad13)
- JP20 pad 14: (no net) -> Net-(JP20-Pad14)
- JP20 pad 15: (no net) -> Net-(JP20-Pad15)
- JP20 pad 16: (no net) -> Net-(JP20-Pad16)
- JP20 pad 17: (no net) -> Net-(JP20-Pad17)
- JP20 pad 18: (no net) -> Net-(JP20-Pad18)
- JP20 pad 19: (no net) -> Net-(JP20-Pad19)
- JP20 pad 2: (no net) -> Net-(JP20-Pad2)
- JP20 pad 3: (no net) -> Net-(JP20-Pad3)
- JP20 pad 4: (no net) -> Net-(JP20-Pad4)
- JP20 pad 5: (no net) -> Net-(JP20-Pad5)
- JP20 pad 6: (no net) -> /GPS_FIX
- JP20 pad 7: (no net) -> Net-(JP20-Pad7)
- JP20 pad 8: (no net) -> Net-(JP20-Pad8)
- JP20 pad 9: (no net) -> /GPS_TX
- JP3 pad 1: (no net) -> GND
- JP7 pad 1: (no net) -> Net-(JP7-Pad1)
- JP7 pad 10: (no net) -> Net-(JP7-Pad10)
- JP7 pad 11: (no net) -> Net-(JP7-Pad11)
- JP7 pad 12: (no net) -> Net-(JP7-Pad12)
- JP7 pad 13: (no net) -> Net-(JP7-Pad13)
- JP7 pad 14: (no net) -> Net-(JP7-Pad14)
- JP7 pad 15: (no net) -> Net-(JP7-Pad15)
- JP7 pad 16: (no net) -> Net-(JP7-Pad16)
- JP7 pad 2: (no net) -> Net-(JP7-Pad2)
- JP7 pad 3: (no net) -> Net-(JP7-Pad3)
- JP7 pad 4: (no net) -> Net-(JP7-Pad4)
- JP7 pad 5: (no net) -> Net-(JP7-Pad5)
- JP7 pad 6: (no net) -> Net-(JP7-Pad6)
- JP7 pad 7: (no net) -> Net-(JP7-Pad7)
- JP7 pad 8: (no net) -> Net-(JP7-Pad8)
- JP7 pad 9: (no net) -> Net-(JP7-Pad9)
- JP9 pad 1: (no net) -> Net-(JP9-Pad1)
- JP9 pad 10: (no net) -> Net-(JP9-Pad10)
- JP9 pad 11: (no net) -> Net-(JP9-Pad11)
- JP9 pad 2: (no net) -> Net-(JP9-Pad2)
- JP9 pad 3: (no net) -> Net-(JP9-Pad3)
- JP9 pad 4: (no net) -> Net-(JP9-Pad4)
- JP9 pad 5: (no net) -> /SDA
- JP9 pad 6: (no net) -> /SCL
- JP9 pad 7: (no net) -> Net-(JP9-Pad7)
- JP9 pad 8: (no net) -> Net-(JP9-Pad8)
- JP9 pad 9: (no net) -> Net-(JP9-Pad9)
- U201 pad 11: (no net) -> Net-(U201-Pad11)
- U201 pad 12: (no net) -> /MPU_INT
- U201 pad 20: (no net) -> Net-(U201-Pad20)
- U201 pad 23: (no net) -> /SCL
- U201 pad 24: (no net) -> /SDA
- U201 pad 7: (no net) -> Net-(U201-Pad7)
- U301 pad 10: (no net) -> /GPS_RX
- U301 pad 13: (no net) -> /GPS_PPS
- U301 pad 14: (no net) -> Net-(U301-Pad14)
- U301 pad 2: (no net) -> Net-(U301-Pad2)
- U301 pad 5: (no net) -> /GPS_FIX
- U301 pad 9: (no net) -> /GPS_TX
- U401 pad 10: (no net) -> Net-(U401-Pad10)
- U401 pad 11: (no net) -> Net-(U401-Pad11)
- U401 pad 13: (no net) -> /SDA
- U401 pad 14: (no net) -> /SCL
- U401 pad 3: (no net) -> Net-(U401-Pad3)
- U401 pad 8: (no net) -> /ADXL_INT
- U401 pad 9: (no net) -> Net-(U401-Pad9)
- U501 pad 1: (no net) -> Net-(U501-Pad1)
- U501 pad 10: (no net) -> Net-(U501-Pad10)
- U501 pad 12: (no net) -> Net-(U501-Pad12)
- U501 pad 13: (no net) -> Net-(U501-Pad13)
- U501 pad 14: (no net) -> /BNO_INT
- U501 pad 19: (no net) -> /SCL
- U501 pad 20: (no net) -> /SDA
- U501 pad 21: (no net) -> Net-(U501-Pad21)
- U501 pad 22: (no net) -> Net-(U501-Pad22)
- U501 pad 23: (no net) -> Net-(U501-Pad23)
- U501 pad 24: (no net) -> Net-(U501-Pad24)
- U501 pad 7: (no net) -> Net-(U501-Pad7)
- U501 pad 8: (no net) -> Net-(U501-Pad8)
- U601 pad 3: (no net) -> /SDA
- U601 pad 4: (no net) -> /SCL
Routing:
- net +3V3: track 0.00 -> 51.8 mm
- net /SDA: track 0.00 -> 31.3 mm
- net /UltimateGPS/VBACKUP: track 0.00 -> 29.0 mm
- net /UltimateGPS/VGPS: track 0.00 -> 14.5 mm
- net /SCL: track 0.00 -> 12.6 mm
- net +5V: track 0.00 -> 5.08 mm
- net +15V: track 0.00 -> 5.08 mm
- net /UltimateGPS/ANT: track 0.00 -> 4.81 mm
- net /BNO055/XOUT32: track 0.00 -> 4.55 mm
- net /HighAcc/VS: track 0.00 -> 4.42 mm
- net /BNO055/XIN32: track 0.00 -> 4.12 mm
- net /GPS_FIX: track 0.00 -> 3.39 mm
- net /GPS_RX: track 0.00 -> 3.32 mm
- net /GPS_TX: track 0.00 -> 2.89 mm
- net /UltimateGPS/VBACKUP+: track 0.00 -> 1.54 mm
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- added copper zone on F.Cu, net GND
Other:
- board outline added: 68.6 x 30.5 mm
- net class Default: clearance 0.2 -> 0.1524; trace_width 0.25 -> 0.1524; via_dia 0.6 -> 0.508; via_drill 0.4 -> 0.3302
- rule pad_to_mask_clearance: 0.2 -> 0
- rule trace_clearance: 0.2 -> 0.1524
- rule trace_min: 0.2 -> 0.1524
- rule via_min_drill: 0.3 -> 0.3302
- rule via_min_size: 0.4 -> 0.508

Commit message: j
Parts:
- added G***: LOGO, KwanSystems:KWAN_CIRCLE_soldermask, F.Cu at (13.0, -6.86)
- added R101: 4k7, KwanSystems:R_Array_Convex_2x0402, F.Cu at (10.2, -15.2)
- added REF**: KiCAD Logo, Symbols:Symbol_KiCAD-Logo_CopperAndSilkScreenTop, B.Cu at (4.06, -15.2)
- added REF**: StKwans, KwanSystems:StKwans, F.Cu at (16.3, -8.13)
- added REF**: StKwans, KwanSystems:ADivisionOf, F.Cu at (17.3, -4.57)
- C503, C509, C525, C526, C528, JP1, JP17, JP2, JP20, JP3, JP4, JP5, JP6, JP7, JP9, U501, Y501: moved to B.Cu
- moved C503 16.1 mm to (17.8, -11.9)
- moved C606 15.1 mm to (20.4, -26.1), turned to 90 degrees
- moved C528 14.8 mm to (21.3, -12.7), turned to 270 degrees
- moved C525 14.8 mm to (22.6, -12.7), turned to 270 degrees
- moved C509 13.1 mm to (15.0, -13.7), turned to 270 degrees
- moved D304 11.7 mm to (55.6, -12.7), turned to 270 degrees
- moved U501 10.8 mm to (17.8, -15.2)
- moved C526 10.4 mm to (23.4, -15.5)
- moved Y501 10.4 mm to (21.3, -15.5), turned to 90 degrees
- moved R304 10.2 mm to (54.4, -12.7), turned to 90 degrees
- moved U601 9.69 mm to (20.2, -23.1), turned to 270 degrees
- moved X311 8.97 mm to (30.7, -13.3), turned to 0 degrees
- moved C208 7.13 mm to (17.8, -11.2)
- moved C210 7.13 mm to (17.8, -12.4)
- moved C213 7.13 mm to (20.6, -15.2)
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Connections:
- JP20 pad 1: Net-(JP20-Pad1) -> (no net)
- JP20 pad 11: Net-(JP20-Pad11) -> (no net)
- JP20 pad 12: Net-(JP20-Pad12) -> (no net)
- JP20 pad 13: Net-(JP20-Pad13) -> (no net)
- JP20 pad 14: Net-(JP20-Pad14) -> (no net)
- JP20 pad 15: Net-(JP20-Pad15) -> (no net)
- JP20 pad 16: Net-(JP20-Pad16) -> (no net)
- JP20 pad 17: Net-(JP20-Pad17) -> (no net)
- JP20 pad 18: Net-(JP20-Pad18) -> (no net)
- JP20 pad 19: Net-(JP20-Pad19) -> (no net)
- JP20 pad 2: Net-(JP20-Pad2) -> (no net)
- JP20 pad 3: Net-(JP20-Pad3) -> (no net)
- JP20 pad 4: Net-(JP20-Pad4) -> (no net)
- JP20 pad 5: Net-(JP20-Pad5) -> (no net)
- JP20 pad 7: Net-(JP20-Pad7) -> (no net)
- JP20 pad 8: Net-(JP20-Pad8) -> (no net)
- JP7 pad 1: Net-(JP7-Pad1) -> (no net)
- JP7 pad 10: Net-(JP7-Pad10) -> (no net)
- JP7 pad 11: Net-(JP7-Pad11) -> (no net)
- JP7 pad 12: Net-(JP7-Pad12) -> /MPU_INT
- JP7 pad 13: Net-(JP7-Pad13) -> (no net)
- JP7 pad 14: Net-(JP7-Pad14) -> (no net)
- JP7 pad 15: Net-(JP7-Pad15) -> (no net)
- JP7 pad 16: Net-(JP7-Pad16) -> (no net)
- JP7 pad 2: Net-(JP7-Pad2) -> (no net)
- JP7 pad 3: Net-(JP7-Pad3) -> (no net)
- JP7 pad 4: Net-(JP7-Pad4) -> /GPS_PPS
- JP7 pad 5: Net-(JP7-Pad5) -> (no net)
- JP7 pad 6: Net-(JP7-Pad6) -> (no net)
- JP7 pad 7: Net-(JP7-Pad7) -> (no net)
- JP7 pad 8: Net-(JP7-Pad8) -> (no net)
- JP7 pad 9: Net-(JP7-Pad9) -> (no net)
- JP9 pad 1: Net-(JP9-Pad1) -> (no net)
- JP9 pad 10: Net-(JP9-Pad10) -> (no net)
- JP9 pad 11: Net-(JP9-Pad11) -> (no net)
- JP9 pad 2: Net-(JP9-Pad2) -> (no net)
- JP9 pad 3: Net-(JP9-Pad3) -> (no net)
- JP9 pad 4: Net-(JP9-Pad4) -> /BNO_INT
- JP9 pad 7: Net-(JP9-Pad7) -> (no net)
- JP9 pad 8: Net-(JP9-Pad8) -> /ADXL_INT
- JP9 pad 9: Net-(JP9-Pad9) -> (no net)
- U201 pad 11: Net-(U201-Pad11) -> (no net)
- U201 pad 20: Net-(U201-Pad20) -> (no net)
- U201 pad 7: Net-(U201-Pad7) -> (no net)
- U301 pad 14: Net-(U301-Pad14) -> (no net)
- U301 pad 2: Net-(U301-Pad2) -> (no net)
- U401 pad 10: Net-(U401-Pad10) -> (no net)
- U401 pad 11: Net-(U401-Pad11) -> (no net)
- U401 pad 3: Net-(U401-Pad3) -> (no net)
- U401 pad 9: Net-(U401-Pad9) -> (no net)
- U501 pad 1: Net-(U501-Pad1) -> (no net)
- U501 pad 10: Net-(U501-Pad10) -> (no net)
- U501 pad 12: Net-(U501-Pad12) -> (no net)
- U501 pad 13: Net-(U501-Pad13) -> (no net)
- U501 pad 21: Net-(U501-Pad21) -> (no net)
- U501 pad 22: Net-(U501-Pad22) -> (no net)
- U501 pad 23: Net-(U501-Pad23) -> (no net)
- U501 pad 24: Net-(U501-Pad24) -> (no net)
- U501 pad 7: Net-(U501-Pad7) -> (no net)
- U501 pad 8: Net-(U501-Pad8) -> (no net)
Routing:
- net +3V3: track 51.8 -> 137.3 mm, vias 0 -> 2
- net /SCL: track 12.6 -> 33.4 mm
- net GND: track 0.00 -> 17.5 mm, vias 0 -> 3
- net /MPU_INT: track 0.00 -> 13.1 mm
- net /UltimateGPS/VGPS: track 14.5 -> 26.1 mm
- net /BNO_INT: track 0.00 -> 10.9 mm
- net /GPS_PPS: track 0.00 -> 10.5 mm
- net /UltimateGPS/VBACKUP: track 29.0 -> 35.9 mm
- net /ADXL_INT: track 0.00 -> 6.33 mm
- net /SDA: track 31.3 -> 36.8 mm, vias 0 -> 2
- net +5V: track 5.08 -> 10.2 mm
- net +15V: track 5.08 -> 10.2 mm
- net /UltimateGPS/ANT: track 4.81 -> 3.21 mm
- added copper zone on B.Cu, net GND
Other:
- board text added: "Designed with"
- board text added: "IOIO Sensinator 01 May 2018"
